File: hw/poetato/di.kicad_sch (KiCad schematic)
At the start: 10 parts, among them Q3 NTK3134N, U12 ISO1211

Commit message: hw: schematic and PCB update
- SE051C2 secure element, ENA tied to 3V3, RST_N to GND
- Epson TSX-3225 24 MHz and FC-135R 32.768 kHz crystals (replace NDK)
- LMR51420 RS-485 5 V buck (replaces TPS54202H)
- Field rail preload removed
- Datasheets updated to match (Würth connector added, unused
  NDK, TPS54202H, IHLP and Murata cap datasheets removed)

Co-Authored-By: Claude Opus 5.5 <noreply@anthropic.com>
Parts:
- U12: Part Number ISO1211 -> ISO1211DR
Other:
- company: (none) -> Jonas Blixt <jonas@blxt.se>
- title: (none) -> PoEtato - Digital input (ISO1211), one channel
Changed lines of the file:
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@@
 	(generator_version "10.0")
 	(paper "A4")
+	(title_block
+		(title "PoEtato - Digital input (ISO1211), one channel")
+		(date "2026-10-08")
+		(rev "A (draft)")
+		(company "Jonas Blixt <jonas@blxt.se>")
+		(comment 1 "Copyright (c) 2026 Jonas Blixt. SPDX-License-Identifier: CERN-OHL-S-2.0")
+		(comment 2 "Licensed under CERN-OHL-S v2: https://ohwr.org/cern_ohl_s_v2.txt")
+		(comment 3 "Source location: https://github.com/jonasblixt/poetato")
+		(comment 4 "Status: draft, not released for manufacture")
+	)
 	(junction
 		(at 96.52 99.06)
@@
 			)
 		)
-		(property "Part Number" "ISO1211"
+		(property "Part Number" "ISO1211DR"
 			(at 26.67 99.314 0)
 			(hide yes)
