File: hw/poetato/do.kicad_sch (KiCad schematic)
At the start: 9 parts, among them K1 AQY212GS, Q1 NTK3134N

Commit message: hw: schematic and PCB update
- SE051C2 secure element, ENA tied to 3V3, RST_N to GND
- Epson TSX-3225 24 MHz and FC-135R 32.768 kHz crystals (replace NDK)
- LMR51420 RS-485 5 V buck (replaces TPS54202H)
- Field rail preload removed
- Datasheets updated to match (Würth connector added, unused
  NDK, TPS54202H, IHLP and Murata cap datasheets removed)

Co-Authored-By: Claude Opus 5.5 <noreply@anthropic.com>
Connections:
- net EN renamed ON
Other:
- company: (none) -> Jonas Blixt <jonas@blxt.se>
- title: (none) -> PoEtato - Digital output (PhotoMOS), one channel
Changed lines of the file:
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@@
 	(generator_version "10.0")
 	(paper "A4")
+	(title_block
+		(title "PoEtato - Digital output (PhotoMOS), one channel")
+		(date "2026-10-08")
+		(rev "A (draft)")
+		(company "Jonas Blixt <jonas@blxt.se>")
+		(comment 1 "Copyright (c) 2026 Jonas Blixt. SPDX-License-Identifier: CERN-OHL-S-2.0")
+		(comment 2 "Licensed under CERN-OHL-S v2: https://ohwr.org/cern_ohl_s_v2.txt")
+		(comment 3 "Source location: https://github.com/jonasblixt/poetato")
+		(comment 4 "Status: draft, not released for manufacture")
+	)
 	(text "< 20ms TtT @ 2.4A"
 		(exclude_from_sim no)
@@
 		)
 	)
-	(hierarchical_label "EN"
+	(hierarchical_label "ON"
 		(shape input)
 		(at 63.5 110.49 180)
