File: hw/poetato/do.kicad_sch (KiCad schematic)
At the start: 9 parts, among them K1 AQY212GS, Q1 NTK3134N

Commit message: hw: name test point nets, debug UART series 1 kOhm, DO notes
- Test point nets named (P12V0_FILTER, POE_VDD, POE_EROUT, VDD_SYS,
  VDD_BAT, VDD_CORE, DCDC_LX, V_SUPERCAP, loop injection nodes, ...)
  (review T4-1)
- R42 330 Ohm -> 1 kOhm on LPUART1_RXD, limits back-feed from a
  USB-UART cable on J4 into an unpowered board (review X2-1)
- DO sheet notes match arch §7: 1.5-2.1 A at a 24 V short (review H4-1)

Co-Authored-By: Claude Opus 5.5 <noreply@anthropic.com>
Other:
- note added: "1.5-2.1 A peak @ 24V short"
- note added: "< 20ms TtT @ 2A"
- note removed: "2.4A peak @ 24V short"
- note removed: "< 20ms TtT @ 2.4A"
Changed lines of the file:
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@@
 		(comment 4 "Status: draft, not released for manufacture")
 	)
-	(text "< 20ms TtT @ 2.4A"
+	(text "< 20ms TtT @ 2A"
 		(exclude_from_sim no)
 		(at 164.846 93.472 0)
@@
 		)
 	)
-	(text "2.4A peak @ 24V short"
+	(text "1.5-2.1 A peak @ 24V short"
 		(exclude_from_sim no)
 		(at 147.32 90.678 0)
