File: hw/poetato/ethernet_poe.kicad_sch (KiCad schematic)
At the start: 106 parts, among them J6 61300211121, T2 FA2672-ALD, T3 7499511440, U3 KSZ8081RNBIA, U4 Si3402-B-GM, U5 VO618A-3X017T, U6 TLVH431AQDBVR, U7 USBLC6-4

Commit message: hw: schematic and PCB update
- SE051C2 secure element, ENA tied to 3V3, RST_N to GND
- Epson TSX-3225 24 MHz and FC-135R 32.768 kHz crystals (replace NDK)
- LMR51420 RS-485 5 V buck (replaces TPS54202H)
- Field rail preload removed
- Datasheets updated to match (Würth connector added, unused
  NDK, TPS54202H, IHLP and Murata cap datasheets removed)

Co-Authored-By: Claude Opus 5.5 <noreply@anthropic.com>
Parts:
- removed C42: ${Capacitance}, Capacitor_SMD:C_0402_1005Metric, symbol cap_mlcc_murata_GRM:GRM/C0402_1u_10V_X7R_10%
- removed C43: ${Capacitance}, Capacitor_SMD:C_0805_2012Metric, symbol cap_mlcc_murata_GRM:GRM/C0805_10u_10V_X7R_10%
- removed R23, R35: 1kΩ, Resistor_SMD:R_0402_1005Metric, symbol res_chip_vishay_crcw:CRCW/R0402_1k0_1_63mW
- added C42: ${Capacitance}, Capacitor_SMD:C_0805_2012Metric, symbol cap_mlcc_murata_GRM:GRM/C0805_22u_6.3V_X7R_20%
- added R35: 4.7kΩ, Resistor_SMD:R_0402_1005Metric, symbol res_chip_vishay_crcw:CRCW/R0402_4k7_1_63mW
- added TP69: TP, TestPoint:TestPoint_Pad_D1.0mm, symbol power:TP
Connections:
- net GND: now also C42.2
- net P3V3: now also C42.1, R35.2
- net POE_VSS2: now also TP69.1
- net at U3.28 (COL/CONFIG0): now also R35.1
Other:
- note added: "Place TP63 on signal without stub. Place TP66 near TP63."
- note added: "TP Placement: - TP4 Close to TP2 (Rectified input voltage measurement) - TP1 Close to TP69 (Switch node measurement) - TP10 Close to TP6 (PD Controller logic supply measurement)"
- company: (none) -> Jonas Blixt <jonas@blxt.se>
- title: (none) -> PoEtato - Ethernet PHY and PoE PD
- moved on the sheet: TP1, TP4
