File: hw/poetato/ethernet_poe.kicad_sch (KiCad schematic)
At the start: 105 parts, among them J6 61300211121, T2 FA2672-ALD, T3 7499511440, U3 KSZ8081RNBIA, U4 Si3402-B-GM, U5 VO618A-3X017T, U6 TLVH431AQDBVR, U7 USBLC6-4

Commit message: hw: name test point nets, debug UART series 1 kOhm, DO notes
- Test point nets named (P12V0_FILTER, POE_VDD, POE_EROUT, VDD_SYS,
  VDD_BAT, VDD_CORE, DCDC_LX, V_SUPERCAP, loop injection nodes, ...)
  (review T4-1)
- R42 330 Ohm -> 1 kOhm on LPUART1_RXD, limits back-feed from a
  USB-UART cable on J4 into an unpowered board (review X2-1)
- DO sheet notes match arch §7: 1.5-2.1 A at a 24 V short (review H4-1)

Co-Authored-By: Claude Opus 5.5 <noreply@anthropic.com>
Connections:
- net POE_VDD: now reaches C55.1, R7.2, TP10.1, U4.3 (VDD)
- net P12V0_FB_1: now reaches R12.1, R14.1, R16.2, TP9.1
- net POE_EROUT: now reaches R30.2, R7.1, TP11.1, U4.1 (EROUT), U5.4
- net P12V0_FILTER: now reaches C57.1, C90.1, L2.1, R16.1, R28.2, TP5.1, TP8.1
Changed lines of the file:
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@@
+		)
+	)
+	(label "P12V0_FILTER"
+		(at 46.99 173.99 0)
+		(effects
+			(font
+				(size 1.27 1.27)
+			)
+			(justify left bottom)
 		)
 	)
@@
 		)
 	)
+	(label "POE_VDD"
+		(at 227.33 219.71 0)
+		(effects
+			(font
+				(size 1.27 1.27)
+			)
+			(justify left bottom)
+		)
+	)
 	(label "POE_VPOS"
 		(at 207.01 186.69 0)
@@
 		)
 	)
+	(label "P12V0_FB_1"
+		(at 55.88 219.71 0)
+		(effects
+			(font
+				(size 1.27 1.27)
+			)
+			(justify left bottom)
+		)
+	)
 	(label "ETH_TX_P"
 		(at 226.06 50.8 0)
@@
 		)
 	)
+	(label "POE_EROUT"
+		(at 161.29 219.71 0)
+		(effects
+			(font
+				(size 1.27 1.27)
+			)
+			(justify left bottom)
+		)
+	)
