File: hw/poetato/ethernet_poe.kicad_sch (KiCad schematic)
At the start: 105 parts, among them J6 61300211121, T2 FA2672-ALD, T3 7499511440, U3 KSZ8081RNBIA, U4 Si3402-B-GM, U5 VO618A-3X017T, U6 TLVH431AQDBVR, U7 USBLC6-4

Commit message: hw: sync symbols with kicadlib field text and value updates
Update Symbols from Library for kicadlib 8686346 (field text 1.27 mm) and
5b35b6c (units on misc R/C values). Value text sizes synced to the library
by script, since a Value reset would also reset power-symbol net names.
Restored BOM_Entry Manufacturer/Part Number and the R57 Power field that the
update cleared, and field positions it reset. Nudged R1, C6, Q6 and C75 text
clear of the larger power-symbol labels. ERC clean, netlist unchanged apart
from the intended values.
Parts:
- C89, C90, C91: value 1nF -> 1.0nF
- R11, R28, R30: value 0 -> 0Ω
- R15: value 12M -> 12MΩ
Other:
- moved on the sheet: R38, R39

Commit message: hw: fix local text collisions and add strap and BOM notes
- MCU: light-pipe note beside D14, TP64/TP65 references off the signal rows
- Ethernet: KSZ8081 strap summary (PHY address 1, RMII, auto-neg 100M),
  TP6 reference clear of POE_VDD
- IO: rating notes merged into the notes box
- DO: PhotoMOS note under K1
- Top level: frame and title around the BOM-only entries

Text and graphics only; ERC clean, netlist unchanged.
Changed lines of the file:
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@@
 		(fields_autoplaced yes)
 		(property "Reference" "TP6"
-			(at 224.79 217.1699 90)
+			(at 219.71 214.63 90)
 			(show_name no)
 			(do_not_autoplace no)
@@
 		)
 	)
+	(text_box "KSZ8081 straps (latched at reset)\nPHYAD = 001: PHY address 1\n   R32, R37 pull-down, R31 pull-up\nCONFIG = 001: RMII\n   R33, R36 pull-down, R35 pull-up\nNWAYEN, SPEED = 1 (R39, R38): auto-neg, 100M\nNAND_Tree# = 1 (R10): normal operation\nDUPLEX, ISO, B-CAST_OFF: internal defaults"
+		(exclude_from_sim no)
+		(at 20.32 27.94 0)
+		(size 55.88 20.32)
+		(margins 0.9525 0.9525 0.9525 0.9525)
+		(stroke
+			(width 0)
+			(type solid)
+		)
+		(fill
+			(type none)
+		)
+		(effects
+			(font
+				(size 1.27 1.27)
+			)
+			(justify left top)
+		)
+	)

Commit message: hw, doc: design rules and impedance net classes
Net classes 50Ohm_RMII, 50Ohm_QSPI, 90Ohm-diff_USB, 100Ohm-diff_MDI,
assigned in the schematic: hidden Netclass fields on the labels, two
rule areas for the PHY-side RMII stubs, ETH_REF_CLK_PHY label after
R26. USB_DP/USB_DM renamed USB_D_P/USB_D_N so KiCad pairs them.

Board rules per doc/pcb-stackup.md section 8: 0.12 mm min track,
0.18 default, 0.15 clearance, vias 0.3/0.6 (0.25/0.45 small), silk and
mask minimums, diff pair presets. poetato.kicad_dru holds the narrower
L3 widths. Unused inner-layer pads removed on all vias. Fab notes:
plain vias, no IPC-4761 Type VII required.
Connections:
- net ETH_REF_CLK_PHY: now reaches R26.2, U3.9 (XI)
Changed lines of the file:
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@@
 			(justify left bottom)
 		)
+		(property "Netclass" "50Ohm_RMII"
+			(at 92.71 83.82 0)
+			(effects
+				(font
+					(size 1.27 1.27)
+					(italic yes)
+				)
+				(justify left)
+				(hide yes)
+			)
+		)
 	)
 	(label "POE_SP1"
@@
 			(justify left bottom)
 		)
+		(property "Netclass" "50Ohm_RMII"
+			(at 92.71 92.71 0)
+			(effects
+				(font
+					(size 1.27 1.27)
+					(italic yes)
+				)
+				(justify left)
+				(hide yes)
+			)
+		)
 	)
 	(label "P12V0_FILTER"
@@
 			(justify left bottom)
 		)
+		(property "Netclass" "100Ohm-diff_MDI"
+			(at 226.06 50.8 0)
+			(effects
+				(font
+					(size 1.27 1.27)
+					(italic yes)
+				)
+				(justify left)
+				(hide yes)
+			)
+		)
 	)
 	(label "ETH_TXD0"
@@
 			(justify left bottom)
 		)
+		(property "Netclass" "50Ohm_RMII"
+			(at 92.71 87.63 0)
+			(effects
+				(font
+					(size 1.27 1.27)
+					(italic yes)
+				)
+				(justify left)
+				(hide yes)
+			)
+		)
 	)
 	(label "POE_SWO"
@@
 			(justify left bottom)
 		)
+		(property "Netclass" "100Ohm-diff_MDI"
+			(at 226.06 53.34 0)
+			(effects
+				(font
+					(size 1.27 1.27)
+					(italic yes)
+				)
+				(justify left)
+				(hide yes)
+			)
+		)
 	)
 	(label "ETH_MDC"
@@
 			(justify left bottom)
 		)
+		(property "Netclass" "50Ohm_RMII"
+			(at 92.71 90.17 0)
+			(effects
+				(font
+					(size 1.27 1.27)
+					(italic yes)
+				)
+				(justify left)
+				(hide yes)
+			)
+		)
 	)
 	(label "ETH_RX_N"
@@
 			(justify left bottom)
 		)
+		(property "Netclass" "100Ohm-diff_MDI"
+			(at 226.06 55.88 0)
+			(effects
+				(font
+					(size 1.27 1.27)
+					(italic yes)
+				)
+				(justify left)
+				(hide yes)
+			)
+		)
 	)
 	(label "POE_CT1"
@@
 			(justify left bottom)
 		)
+		(property "Netclass" "50Ohm_RMII"
+			(at 92.71 71.12 0)
+			(effects
+				(font
+					(size 1.27 1.27)
+					(italic yes)
+				)
+				(justify left)
+				(hide yes)
+			)
+		)
 	)
 	(label "ETH_LED1_ACT_N"
@@
 			(justify left bottom)
 		)
+		(property "Netclass" "100Ohm-diff_MDI"
+			(at 226.06 48.26 0)
+			(effects
+				(font
+					(size 1.27 1.27)
+					(italic yes)
+				)
+				(justify left)
+				(hide yes)
+			)
+		)
 	)
 	(label "ETH_RXD0"
@@
 			(justify left bottom)
 		)
+		(property "Netclass" "50Ohm_RMII"
+			(at 92.71 68.58 0)
+			(effects
+				(font
+					(size 1.27 1.27)
+					(italic yes)
+				)
+				(justify left)
+				(hide yes)
+			)
+		)
 	)
 	(label "ETH_REF_CLK"
@@
 			(justify left bottom)
 		)
+		(property "Netclass" "50Ohm_RMII"
+			(at 92.71 139.7 0)
+			(effects
+				(font
+					(size 1.27 1.27)
+					(italic yes)
+				)
+				(justify left)
+				(hide yes)
+			)
+		)
 	)
 	(label "ETH_LED0_LINK_N"
@@
 			)
 		)
+	)
+	(rule_area
+		(polyline
+			(pts
+				(xy 133.35 69.85) (xy 129.54 69.85) (xy 129.54 74.93) (xy 133.35 74.93)
+			)
+			(stroke
+				(width 0)
+				(type dash)
+			)
+			(fill
+				(type none)
+			)
+		)
+	)
+	(netclass_flag ""
+		(length 2.54)
+		(shape round)
+		(at 130.81 69.85 0)
+		(effects
+			(font
+				(size 1.27 1.27)
+			)
+			(justify left bottom)
+		)
+		(property "Netclass" "50Ohm_RMII"
+			(at 129.794 67.31 0)
+			(effects
+				(font
+					(size 1.27 1.27)
+					(italic yes)
+				)
+				(justify right)
+			)
+		)
+	)
+	(rule_area
+		(polyline
+			(pts
+				(xy 133.35 85.09) (xy 129.54 85.09) (xy 129.54 96.52) (xy 133.35 96.52)
+			)
+			(stroke
+				(width 0)
+				(type dash)
+			)
+			(fill
+				(type none)
+			)
+		)
+	)
+	(netclass_flag ""
+		(length 2.54)
+		(shape round)
+		(at 130.81 96.52 180)
+		(effects
+			(font
+				(size 1.27 1.27)
+			)
+			(justify right bottom)
+		)
+		(property "Netclass" "50Ohm_RMII"
+			(at 129.794 99.06 0)
+			(effects
+				(font
+					(size 1.27 1.27)
+					(italic yes)
+				)
+				(justify right)
+			)
+		)
+	)
+	(label "ETH_REF_CLK_PHY"
+		(at 130.81 142.24 0)
+		(effects
+			(font
+				(size 1.27 1.27)
+			)
+			(justify left bottom)
+		)
+		(property "Netclass" "50Ohm_RMII"
+			(at 130.81 139.7 0)
+			(effects
+				(font
+					(size 1.27 1.27)
+					(italic yes)
+				)
+				(justify left)
+				(hide yes)
+			)
+		)
