File: hw/poetato/io.kicad_sch (KiCad schematic)
At the start: 40 parts, among them J1 1757349, J2 1757268, Q6 NTK3134N, T1 1308_750319693, U15 SN6507DGQR, U19 TPS26625DRCR

Commit message: hw: schematic and PCB update
- SE051C2 secure element, ENA tied to 3V3, RST_N to GND
- Epson TSX-3225 24 MHz and FC-135R 32.768 kHz crystals (replace NDK)
- LMR51420 RS-485 5 V buck (replaces TPS54202H)
- Field rail preload removed
- Datasheets updated to match (Würth connector added, unused
  NDK, TPS54202H, IHLP and Murata cap datasheets removed)

Co-Authored-By: Claude Opus 5.5 <noreply@anthropic.com>
Parts:
- removed C34: ${Capacitance}, Capacitor_SMD:C_0603_1608Metric, symbol cap_mlcc_murata_GRM:GRM/C0603_2u2_10V_X7R_10%
- removed R8: 10kΩ, Resistor_SMD:R_1206_3216Metric, symbol res_chip_vishay_crcw:CRCW/R1206_10k0_1_250mW
- added C34: ${Capacitance}, Capacitor_SMD:C_0603_1608Metric, symbol cap_mlcc_murata_GRM:GRM/C0603_4u7_10V_X7R_10%
- added TP67, TP68: TP, TestPoint:TestPoint_Pad_D1.0mm, symbol power:TP
- U15: Part Number SN6507DGQR -> SN6507DGQR
Connections:
- net RS485/RS485_SIGNAL_GND is gone; now on net GND_FIELD: J2.3
- net GND: now also C34.2, TP68.1
- net GND_FIELD: now also TP67.1
- net at R72.1, U15.8 (SS/ILIM): now also C34.1
- net DO1_EN renamed DO1_ON
- net DO2_EN renamed DO2_ON
- net RS485/RS485_SHIELD renamed SHIELD
Other:
- sheet Digital Output ports: added ON; removed EN
- sheet Digital Output1 ports: added ON; removed EN
- sheet RS485 ports: added none; removed RS485_SHIELD, RS485_SIGNAL_GND
- note added: "Isolated 24V, 3W supply"
- note added: "Output 1 - 2: ≤ 30 V DC, ≤ 17 V AC rms (≤ 48 V peak-to-peak), 100mA, dry contact OptoMOS outputs"
- note removed: "Isolated 24V, 1.5W supply"
- note removed: "Output 1 - 2: 60V AC/DC, 1A, dry contact OptoMOS outputs"
- company: (none) -> Jonas Blixt <jonas@blxt.se>
- title: (none) -> PoEtato - Field I/O, isolated 24 V supply
