File: hw/poetato/io.kicad_sch (KiCad schematic)
At the start: 16 parts, among them J1 1757349, J2 1757268, U19 TPS26625DRCR

Commit message: hw: fix local text collisions and add strap and BOM notes
- MCU: light-pipe note beside D14, TP64/TP65 references off the signal rows
- Ethernet: KSZ8081 strap summary (PHY address 1, RMII, auto-neg 100M),
  TP6 reference clear of POE_VDD
- IO: rating notes merged into the notes box
- DO: PhotoMOS note under K1
- Top level: frame and title around the BOM-only entries

Text and graphics only; ERC clean, netlist unchanged.
Other:
- note removed: "Input 1 - 3: IEC 61131-2, Type 3 Sinking inputs"
- note removed: "Output 1 - 2: ≤ 30 V DC, 100mA, dry contact OptoMOS outputs"
Changed lines of the file:
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@@
 		(comment 4 "Status: draft, not released for manufacture")
-	)
-	(text "Output 1 - 2: ≤ 30 V DC, 100mA, dry contact OptoMOS outputs"
-		(exclude_from_sim no)
-		(at 352.552 140.462 0)
-		(effects
-			(font
-				(size 1.27 1.27)
-			)
-		)
 	)
 	(text "Isolation barrier"
@@
 		)
 	)
-	(text "Input 1 - 3: IEC 61131-2, Type 3 Sinking inputs"
-		(exclude_from_sim no)
-		(at 347.218 167.132 0)
-		(effects
-			(font
-				(size 1.27 1.27)
-			)
-		)
-	)
-	(text_box "Isolation:\n\nOutput 1 - 2 are Isolated from each other and the logic\n\nInput 1 - 3 are Isolated from each other and the logic\n\n24V Field supply is isolated from logic but powers isolated sides of RS485"
+	(text_box "Isolation:\n\nOutput 1 - 2 are Isolated from each other and the logic\n\nInput 1 - 3 are Isolated from each other and the logic\n\n24V Field supply is isolated from logic but powers isolated sides of RS485\n\nRatings:\n\nOutput 1 - 2: ≤ 30 V DC, 100mA, dry contact OptoMOS outputs\n\nInput 1 - 3: IEC 61131-2, Type 3 Sinking inputs"
 		(exclude_from_sim no)
 		(at 334.01 113.54 0)
-		(size 55.88 22.35)
+		(size 55.88 38.1)
 		(margins 0.9525 0.9525 0.9525 0.9525)
 		(stroke
