File: hw/poetato/mcu.kicad_sch (KiCad schematic)
At the start: 102 parts, among them J3 FTSH-105-01-L-DV-007-K, J4 61300611121, Q10 NTK3134N, Q9 NTK3134N, U1 MCXN247VKLT, U10 SE051, U11 S25FL064LABMFI013, U18 TPS563252DRLR, U2 LP3470A293DBVR, U8 USBLC6-4, U9 USBLC6-4, Y1 32.768kHz, Y3 24MHz

Commit message: hw: schematic and PCB update
- SE051C2 secure element, ENA tied to 3V3, RST_N to GND
- Epson TSX-3225 24 MHz and FC-135R 32.768 kHz crystals (replace NDK)
- LMR51420 RS-485 5 V buck (replaces TPS54202H)
- Field rail preload removed
- Datasheets updated to match (Würth connector added, unused
  NDK, TPS54202H, IHLP and Murata cap datasheets removed)

Co-Authored-By: Claude Opus 5.5 <noreply@anthropic.com>
Parts:
- removed C1, C2: ${Capacitance}, Capacitor_SMD:C_0402_1005Metric, symbol cap_mlcc_murata_GRM:GRM/C0402_4p7_50V_C0G_0.1pF
- removed Y1: 32.768kHz, Jonas:NX3215SA, symbol xtal_ndk:NDK/NX3215SA-32.768K-STD-MUA-8
- removed Y3: 24MHz, Jonas:NX3225SA, symbol xtal_ndk:NDK/NX3225SA-24.000MHZ-STD-CSR-1
- added C1, C2: ${Capacitance}, Capacitor_SMD:C_0402_1005Metric, symbol cap_mlcc_murata_GRM:GRM/C0402_10p_50V_C0G_2%
- added C43: ${Capacitance}, Capacitor_SMD:C_0402_1005Metric, symbol cap_mlcc_murata_GRM:GRM/C0402_1u_10V_X7R_10%
- added J8: 614105150721, Connector_USB:USB_Micro-B_Wuerth_614105150721_Vertical, symbol connectors:Wurth_614105150721
- added U20: USBLC6-4, Package_TO_SOT_SMD:SOT-23-6, symbol diode_misc:USBLC6-4
- added Y1: 32.768kHz, Jonas:NX3215SA, symbol xtal_epson:Epson/X1A0001410006
- added Y3: 24MHz, Jonas:NX3225SA, symbol xtal_epson:Epson/X1E0000210048
Connections:
- net GND: now also C1.2, C2.2, C43.2, J8.5, J8.SH, U20.2 (GND), Y3.2 (G), Y3.4 (G)
- net at C4.1, U1.49 (P5_1/XTAL32K): now also Y1.2
- net at U1.11 (P1_31/EXTAL48M): now also C2.1, Y3.3
- net at U1.10 (P1_30/XTAL48M): now also C1.1, Y3.1
- net USB_DP: now reaches U1.40 (USB1_DP)
- net USB_DP: now also J8.3, U20.6 (IO4)
- net USB_DM: now reaches U1.41 (USB1_DM)
- net USB_DM: now also J8.2, U20.4 (IO3)
- net USB_VBUS: now reaches U1.42 (USB1_VBUS)
- net USB_VBUS: now also C43.1, J8.1, U20.5 (VBUS)
- net at C3.1, U1.48 (P5_0/EXTAL32K): now also Y1.1
Other:
- note added: "MCU has internal, controllable load caps. These are backup if we need more."
- note added: "Place TP64 on signal without stub. Place TP65 near TP64."
- note added: "RTC & SRAM Backup power (>= 8h)"
- note removed: "RTC & SRAM Backup power (~24h)"
- note removed: "TODO: Add HS USB"
- company: (none) -> Jonas Blixt <jonas@blxt.se>
- title: (none) -> PoEtato - MCU, secure element, flash and 3.3 V supply
