File: hw/poetato/mcu.kicad_sch (KiCad schematic)
At the start: 105 parts, among them J3 FTSH-105-01-L-DV-007-K, J4 61300611121, J8 614105150721, Q10 NTK3134N, Q9 NTK3134N, U1 MCXN247VKLT, U10 SE051, U11 S25FL064LABMFI013, U18 TPS563252DRLR, U2 LP3470A293DBVR, U20 USBLC6-4, U8 USBLC6-4, U9 USBLC6-4, Y1 32.768kHz, Y3 24MHz

Commit message: hw: RS485_RXD pull-up, 3V3 buck EN threshold, DC-only output rating
- R8 100 kOhm pull-up from RS485_RXD to P3V3 (review X3-1)
- 3V3 buck EN divider R23 127 kOhm / R87 20.5 kOhm (replaces R86
  47 kOhm): on at ~8.6 V, off at ~7.2 V (review Q-4)
- IO sheet note: outputs rated <= 30 V DC only (review E1-1)

Co-Authored-By: Claude Opus 5.5 <noreply@anthropic.com>
Parts:
- removed R86: 47kΩ, Resistor_SMD:R_0402_1005Metric, symbol res_chip_vishay_crcw:CRCW/R0402_47k0_1_63mW
- added R23: 127kΩ, Resistor_SMD:R_0402_1005Metric, symbol res_chip_vishay_crcw:CRCW/R0402_127k0_1_63mW
Connections:
- net P12V0: now also R23.1
- net P3V3: now also D17.3 (common)
- net at C33.1, R50.1, TP16.1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: now also D17.2 (K); no longer D17.3 (K)
- net at C81.1, R87.1, U18.5 (EN): now also R23.2

Commit message: hw: name test point nets, debug UART series 1 kOhm, DO notes
- Test point nets named (P12V0_FILTER, POE_VDD, POE_EROUT, VDD_SYS,
  VDD_BAT, VDD_CORE, DCDC_LX, V_SUPERCAP, loop injection nodes, ...)
  (review T4-1)
- R42 330 Ohm -> 1 kOhm on LPUART1_RXD, limits back-feed from a
  USB-UART cable on J4 into an unpowered board (review X2-1)
- DO sheet notes match arch §7: 1.5-2.1 A at a 24 V short (review H4-1)

Co-Authored-By: Claude Opus 5.5 <noreply@anthropic.com>
Parts:
- removed R42, R43: 330Ω, Resistor_SMD:R_0402_1005Metric, symbol res_chip_vishay_crcw:CRCW/R0402_330R0_1_63mW
- added R42, R43: 1kΩ, Resistor_SMD:R_0402_1005Metric, symbol res_chip_vishay_crcw:CRCW/R0402_1k0_1_63mW
- added TP70: TP, TestPoint:TestPoint_Pad_D1.0mm, symbol power:TP
Connections:
- net GND: now also TP70.1
- net LPUART1_RXD: now also R42.2
- net LPUART1_TXD: now also R43.2
- net VDD_BAT: now reaches C33.1, D17.2 (K), R50.1, TP16.1, U1.47 (VDD_BAT)
- net V_SUPERCAP: now reaches C9.1, R50.2, TP36.1
- net VDD_CORE: now reaches C19.1, C20.1, C21.1, C22.1, L1.2, TP17.1, U1.12 (VDD_CORE), U1.58 (VDD_CORE)
- net at J4.5, U9.1 (IO1): now also R43.1
- net at J4.4, U9.4 (IO3): now also R42.1
- net P3V3_FB: now reaches C84.2, R63.2, R89.1, U18.6 (FB)
- net DCDC_LX: now reaches L1.1, TP18.1, U1.53 (DCDC_LX)
- net VDD_SYS: now reaches C18.1, TP13.1, U1.55 (VDD_SYS)
- net P3V3_FB_1: now reaches C84.1, R63.1, R88.2, TP22.1
Other:
- note added: "TP18/TP70 Switch node measurement"
- moved on the sheet: R50, TP22, TP36
