File: hw/poetato/poetato.kicad_pcb (KiCad board)
At the start: 6 copper layers, 139 x 87 mm, 308 parts, among them J1 1757349, J2 1757268, J3 FTSH-105-01-L-DV-007-K, J4 61300611121, J5 61300211121, K1 AQY212GS, K2 AQY212GS, Q1 NTK3134N, Q10 NTK3134N, Q11 NTK3134N, Q12 NTK3134N, Q13 NTK3134N, Q3 NTK3134N, Q6 NTK3134N, Q7 FDV304P, Q8 FDV304P, Q9 NTK3134N, T1 1308_750319693, T2 FA2672-ALD, T3 7499511440, U1 MCXN247VKLT, U10 SE051, U11 S25FL064LABMFI013, U12 ISO1211, U13 ISO1211, U14 ISO1211, U15 SN6507DGQR, U16 ISO3082, U17 TPS54202HDDCR, U18 TPS563252DRLR, U2 LP3470A293DBVR, U3 KSZ8081RNBIA, U4 Si3402-B-GM, U5 VO618A-3X017T, U6 TLVH431AQDBVR, U7 USBLC6-4, U8 USBLC6-4, U9 USBLC6-4, Y1 32.768kHz, Y3 24MHz

Commit message: hw: schematic and PCB update
- SE051C2 secure element, ENA tied to 3V3, RST_N to GND
- Epson TSX-3225 24 MHz and FC-135R 32.768 kHz crystals (replace NDK)
- LMR51420 RS-485 5 V buck (replaces TPS54202H)
- Field rail preload removed
- Datasheets updated to match (Würth connector added, unused
  NDK, TPS54202H, IHLP and Murata cap datasheets removed)

Co-Authored-By: Claude Opus 5.5 <noreply@anthropic.com>
Parts:
- removed C70: 1nF, Jonas:C_Murata_GA3_5.7x2.8
- removed F4: 390mA, Jonas:FUSC3216X85N
- removed R8: 10kΩ, Resistor_SMD:R_1206_3216Metric
- added C89: 1nF, Capacitor_SMD:C_1808_4520Metric, F.Cu at (38.6, 126.9)
- added C90: 1nF, Capacitor_SMD:C_1808_4520Metric, F.Cu at (38.6, 130.8)
- added C91: 1nF, Capacitor_SMD:C_1808_4520Metric, F.Cu at (38.6, 134.6)
- added C92: 1nF, Capacitor_SMD:C_1808_4520Metric, F.Cu at (47.9, 126.9)
- added C93: 4.7uF, Capacitor_SMD:C_1206_3216Metric, F.Cu at (220.1, 134.5)
- added J6: 61300211121, Connector_PinHeader_2.54mm:PinHeader_1x02_P2.54mm_Vertical, F.Cu at (168.8, 141.8)
- added J8: 614105150721, Connector_USB:USB_Micro-B_Wuerth_614105150721_Vertical, F.Cu at (88.2, 37.8)
- added R51: 200kΩ, Resistor_SMD:R_0603_1608Metric, F.Cu at (33.2, 82.1)
- added R85: 14kΩ, Resistor_SMD:R_0603_1608Metric, F.Cu at (42.0, 74.2)
- added R95: 100kΩ, Resistor_SMD:R_0603_1608Metric, F.Cu at (33.9, 85.1)
- added R97: 100kΩ, Resistor_SMD:R_0402_1005Metric, F.Cu at (215.9, 138.4)
- added TP50: TP, TestPoint:TestPoint_Pad_D1.0mm, F.Cu at (182.8, 141.1)
- added TP51: TP, TestPoint:TestPoint_Pad_D1.0mm, F.Cu at (165.0, 141.1)
- added TP52: TP, TestPoint:TestPoint_Pad_D1.0mm, F.Cu at (165.0, 144.1)
- added TP53: TP, TestPoint:TestPoint_Pad_D1.0mm, F.Cu at (165.0, 147.2)
- added TP54: TP, TestPoint:TestPoint_Pad_D1.0mm, F.Cu at (165.0, 150.2)
- added TP55: TP, TestPoint:TestPoint_Pad_D1.0mm, F.Cu at (174.7, 141.1)
- added TP56: TP, TestPoint:TestPoint_Pad_D1.0mm, F.Cu at (174.7, 144.1)
- added TP57: TP, TestPoint:TestPoint_Pad_D1.0mm, F.Cu at (174.7, 147.2)
- added TP58: TP, TestPoint:TestPoint_Pad_D1.0mm, F.Cu at (174.7, 150.2)
- added TP59: TP, TestPoint:TestPoint_Pad_D1.0mm, F.Cu at (177.7, 141.1)
- added TP60: TP, TestPoint:TestPoint_Pad_D1.0mm, F.Cu at (177.7, 144.1)
- added TP61: TP, TestPoint:TestPoint_Pad_D1.0mm, F.Cu at (177.7, 147.2)
- added TP62: TP, TestPoint:TestPoint_Pad_D1.0mm, F.Cu at (95.6, 165.0)
- added TP63: TP, TestPoint:TestPoint_Pad_D1.0mm, F.Cu at (95.6, 168.1)
- added TP64: TP, TestPoint:TestPoint_Pad_D1.0mm, F.Cu at (100.7, 165.0)
- added TP65: TP, TestPoint:TestPoint_Pad_D1.0mm, F.Cu at (100.7, 168.1)
- added TP66: TP, TestPoint:TestPoint_Pad_D1.0mm, F.Cu at (95.6, 171.1)
- added TP67: TP, TestPoint:TestPoint_Pad_D1.0mm, F.Cu at (201.5, 61.5)
- added TP68: TP, TestPoint:TestPoint_Pad_D1.0mm, F.Cu at (201.5, 64.6)
- added TP69: TP, TestPoint:TestPoint_Pad_D1.0mm, F.Cu at (192.0, 64.6)
- added U19: TPS26625DRCR, Package_SON:VSON-10-1EP_3x3mm_P0.5mm_EP1.65x2.4mm, F.Cu at (37.6, 88.9)
- added U20: USBLC6-4, Package_TO_SOT_SMD:SOT-23-6, F.Cu at (196.0, 54.5)
- C1, C2: value 4.7pF -> 10.0pF
- C34: value 2.2uF -> 4.7uF
- C42: value 1.0uF -> 22.0uF; footprint Capacitor_SMD:C_0402_1005Metric -> Capacitor_SMD:C_0805_2012Metric
- C43: value 10.0uF -> 1.0uF; footprint Capacitor_SMD:C_0805_2012Metric -> Capacitor_SMD:C_0402_1005Metric
- C52: value 1nF -> 1.0uF; footprint Jonas:C_Murata_GA3_5.7x2.8 -> Capacitor_SMD:C_0805_2012Metric
- C53, C58: value 1nF -> 1.0uF; footprint Jonas:C_Murata_GA3_5.7x2.8 -> Capacitor_SMD:C_1206_3216Metric
- C76, C77: footprint Capacitor_SMD:C_0402_1005Metric -> Capacitor_SMD:C_0805_2012Metric
- C80: value 10.0uF -> 4.7uF; footprint Capacitor_SMD:C_0805_2012Metric -> Capacitor_SMD:C_1206_3216Metric
- D18, D19: value 31.1V -> 36.7V
- L3: value 22µH -> 10µH
- R35: value 1kΩ -> 4.7kΩ
- R82: value 13.3kΩ -> 13.7kΩ
- R83: value 510kΩ -> 1MΩ
- U17: value TPS54202HDDCR -> LMR51420XDDCR
- moved C34 172.2 mm to (205.1, 61.2), turned to 0 degrees
- moved D18 135.8 mm to (177.7, 135.3), turned to 0 degrees
- moved L5 133.3 mm to (33.7, 88.4), turned to 90 degrees
- moved TP48 131.8 mm to (233.6, 109.9)
- moved TP49 131.8 mm to (233.6, 112.9)
- moved TP31 129.2 mm to (227.5, 112.9)
- moved TP46 126.1 mm to (230.6, 109.9)
- moved TP47 126.1 mm to (230.6, 112.9)
- moved TP27 124.6 mm to (227.5, 109.9)
- moved D24 124.1 mm to (38.5, 93.0)
- moved U16 120.6 mm to (227.8, 102.4)
- moved D19 116.7 mm to (167.6, 135.3), turned to 0 degrees
- moved D27 113.4 mm to (213.3, 98.6)
- moved Q7 113.4 mm to (213.3, 103.1)
- moved Q8 113.4 mm to (213.3, 107.5)
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Connections:
- C43 pad 1: P3V3 -> /MCU/USB_VBUS
- C52 pad 1: GND -> Net-(U19-dVdT)
- C52 pad 2: /Ethernet & PoE/POE_VNEG -> Net-(U19-OVP)
- C53 pad 1: Net-(C53-Pad1) -> P24V0_FIELD
- C53 pad 2: /Ethernet & PoE/POE_VPOS -> GND_FIELD
- C57 pad 1: Net-(C53-Pad1) -> Net-(C57-Pad1)
- C58 pad 1: SHIELD -> /IO/P24V0_FIELD_PROT
- C58 pad 2: GND -> GND_FIELD
- L2 pad 1: Net-(C53-Pad1) -> Net-(C57-Pad1)
- R16 pad 1: Net-(C53-Pad1) -> Net-(C57-Pad1)
- R28 pad 2: Net-(C53-Pad1) -> Net-(C57-Pad1)
- TP5 pad 1: Net-(C53-Pad1) -> Net-(C57-Pad1)
- TP8 pad 1: Net-(C53-Pad1) -> Net-(C57-Pad1)
- U1 pad 40: unconnected-(U1-USB1_DP-Pad40) -> /MCU/USB_DP
- U1 pad 41: unconnected-(U1-USB1_DM-Pad41) -> /MCU/USB_DM
- U1 pad 42: unconnected-(U1-USB1_VBUS-Pad42) -> /MCU/USB_VBUS
Routing:
- net Net-(C57-Pad1): track 0.00 -> 40.8 mm
- net Net-(C53-Pad1): track 40.8 -> 0.00 mm
- net GND_FIELD: track 16.9 -> 0.00 mm
- net Net-(D23-A): track 14.6 -> 0.00 mm
- net (no net): track 40.7 -> 27.3 mm
- net /IO/P24V0_FIELD_PROT: track 13.2 -> 0.00 mm
- net Net-(D25-A): track 11.6 -> 0.00 mm
- net Net-(D7-Pad1): track 10.2 -> 0.00 mm
- net Net-(D23-K): track 4.82 -> 0.00 mm
- net Net-(D7-Pad2): track 4.03 -> 0.00 mm
- net Net-(C71-Pad2): track 2.49 -> 0.00 mm
- net Net-(C36-Pad2): track 2.49 -> 0.00 mm
- net /MCU/DO1_ON: track 2.85 -> 0.85 mm
- net Net-(K1-Pad1): track 1.75 -> 0.00 mm
- net GND: track 72.4 -> 71.2 mm, vias 92 -> 91
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