File: hw/poetato/poetato.kicad_pcb (KiCad board)
At the start: 6 copper layers, 139 x 87 mm, 338 parts, among them J1 1757349, J2 1757268, J3 FTSH-105-01-L-DV-007-K, J4 61300611121, J5 61300211121, J6 61300211121, J8 614105150721, K1 AQY212GS, K2 AQY212GS, Q1 NTK3134N, Q10 NTK3134N, Q11 NTK3134N, Q12 NTK3134N, Q13 NTK3134N, Q3 NTK3134N, Q6 NTK3134N, Q7 FDV304P, Q8 FDV304P, Q9 NTK3134N, T1 1308_750319693, T2 FA2672-ALD, T3 7499511440, U1 MCXN247VKLT, U10 SE051, U11 S25FL064LABMFI013, U12 ISO1211, U13 ISO1211, U14 ISO1211, U15 SN6507DGQR, U16 ISO3082, U17 LMR51420XDDCR, U18 TPS563252DRLR, U19 TPS26625DRCR, U2 LP3470A293DBVR, U20 USBLC6-4, U3 KSZ8081RNBIA, U4 Si3402-B-GM, U5 VO618A-3X017T, U6 TLVH431AQDBVR, U7 USBLC6-4, U8 USBLC6-4, U9 USBLC6-4, Y1 32.768kHz, Y3 24MHz

Commit message: hw, doc: JLC06161H-2116A stackup and impedance classes
Stackup drawing and controlled-impedance table on User.3 (named
User.Stackup), right of the board. New doc/pcb-stackup.md with the
stackup, why 2116A, the 50/90/100 ohm classes and routing rules;
doc/scripts/impedance.py is the 2D field solver behind the widths.
Decision log row, verification-plan check of the fab impedance report.
Other:
- board text added: "-"
- board text added: "0.0152 mm"
- board text added: "0.0350 mm"
- board text added: "0.1164 mm"
- board text added: "0.12"
- board text added: "0.13"
- board text added: "0.13 mm"
- board text added: "0.14"
- board text added: "0.15"
- board text added: "0.16"
- board text added: "0.18"
- board text added: "0.20"
- board text added: "0.70 mm"
- board text added: "1. Widths from a 2D field solve: solder mask Dk 3.8, 30 µm over laminate, 15 µm over Cu;"
- board text added: "100 Ω diff"
- board text added: "2. L3 references L2 GND (0.13 mm); L4 PWR is 0.93 mm away. Route L3 signals only"
- board text added: "3. Dk per JLCPCB: prepreg 2116 4.16, core 4.6."
- board text added: "4.16"
- board text added: "4.60"
- board text added: "50 Ω SE"
- board text added: "6 layers, 1.6 mm finished (1.556 mm laminate + mask), outer 1 oz, inner 0.5 oz, FR-4"
- board text added: "90 Ω diff"
- board text added: "B.Cu"
- board text added: "CONTROLLED IMPEDANCE (order with impedance control)"
- board text added: "Copper 0.5 oz"
- board text added: "Copper 1 oz"
- board text added: "Core"
- board text added: "Core, no Cu"
- board text added: "Cross-section (vertical x28)"
- board text added: "Dk"
- board text added: "ETH_TX_P/N, ETH_RX_P/N"
- board text added: "F.Cu"
- board text added: "Geometry"
- board text added: "H = dielectric to reference"
- board text added: "In1.Cu"
- board text added: "In2.Cu"
- board text added: "In3.Cu"
- board text added: "In4.Cu"
- board text added: "L1 / L6"
- board text added: "L1 SIG"
- board text added: "L2 / L5 GND"
- board text added: "L2 GND"
- board text added: "L3"
- board text added: "L3 SIG"
- board text added: "L4 PWR"
- board text added: "L5 GND"
- board text added: "L6 SIG"
- board text added: "Layer"
- board text added: "Material"
- board text added: "Notes"
- board text added: "PCB STACKUP JLCPCB JLC06161H-2116A"
- board text added: "Prepreg 2116"
- board text added: "RMII, ETH_REF_CLK, QSPI"
- board text added: "Reference"
- board text added: "Reference plane (GND)"
- board text added: "S"
- board text added: "S mm"
- board text added: "SE: one trace of width W"
- board text added: "Signals"
- board text added: "Target"
- board text added: "Thickness"
- board text added: "Total 1.556 mm (+ solder mask, Dk 3.8)"
- board text added: "USB_DP / USB_DM"
- board text added: "Use"
- board text added: "W"
- board text added: "W mm"
- board text added: "calculator for JLC06161H-2116A before ordering."
- board text added: "over unbroken L2 GND."
- board text added: "rectangular trace profile. Expect about ±5 %. Confirm in the JLCPCB impedance"

Commit message: hw, doc: vendor-neutral fab requirements, physical stackup in Board Setup
Board Setup now holds the JLC06161H-2116A stackup (impedance controlled,
ENIG, LPI mask Dk 3.8), so the Gerber job, IPC-2581 and ODB++ exports
carry it. Fabrication notes on User.Stackup below the board, and
doc/pcb-stackup.md §7 with the same requirements: IPC-6012 Class 2,
Tg >= 150, 1.60 mm +-10 %, finished copper, impedance +-10 % with
coupons and report, the dielectric gaps another fab must keep.
doc/scripts/stackup_drawing.py regenerates the drawing.
Other:
- board text added: "1. Build to IPC-6012 Class 2. 6-layer rigid FR-4, Tg >= 150 °C, rated for lead-free assembly."
- board text added: "2. Finished board thickness 1.60 mm ±10 %."
- board text added: "3. Dk per JLCPCB: prepreg 2116 4.16, core 4.6 (test frequency not stated)."
- board text added: "3. Finished copper: outer layers 1 oz (35 µm), inner layers 0.5 oz."
- board text added: "4. Layer order and use per the stackup table. Dielectric thicknesses are nominal; other materials and"
- board text added: "5. Controlled impedance per the table, ±10 %. The fab may change the width of controlled traces by up to"
- board text added: "6. Surface finish ENIG. LPI solder mask both sides, Dk about 3.8."
- board text added: "FABRICATION NOTES"
- board text added: "L1-L2, L2-L3, L4-L5 and L5-L6 each stay <= 0.15 mm."
- board text added: "Reference build: JLCPCB stackup JLC06161H-2116A, Tg 155 option."
- board text added: "constructions are acceptable if the impedance targets and finished thickness are met and"
- board text added: "report are required (IPC-TM-650 2.5.5.7)."
- board text added: "±0.025 mm (keeping the pair pitch) to meet the targets. TDR test coupons and an impedance test"
- board text removed: "3. Dk per JLCPCB: prepreg 2116 4.16, core 4.6."

Commit message: hw, doc: design rules and impedance net classes
Net classes 50Ohm_RMII, 50Ohm_QSPI, 90Ohm-diff_USB, 100Ohm-diff_MDI,
assigned in the schematic: hidden Netclass fields on the labels, two
rule areas for the PHY-side RMII stubs, ETH_REF_CLK_PHY label after
R26. USB_DP/USB_DM renamed USB_D_P/USB_D_N so KiCad pairs them.

Board rules per doc/pcb-stackup.md section 8: 0.12 mm min track,
0.18 default, 0.15 clearance, vias 0.3/0.6 (0.25/0.45 small), silk and
mask minimums, diff pair presets. poetato.kicad_dru holds the narrower
L3 widths. Unused inner-layer pads removed on all vias. Fab notes:
plain vias, no IPC-4761 Type VII required.
Other:
- board text added: "7. Vias are plain plated through-holes, smallest finished hole 0.25 mm. No via filling or capping"
- board text added: "USB_D_P / USB_D_N"
- board text added: "required (no IPC-4761 Type VII). Non-functional inner-layer pads are removed in the data."
- board text removed: "USB_DP / USB_DM"

Commit message: hw, doc: SWD as 50 ohm controlled impedance
New net class 50Ohm_SWD (0.18 mm outer, 0.16 mm on L3 via the .kicad_dru
rule) for SWDCLK, SWDIO and SWO, assigned by a rule area on the MCU
sheet. MCX N247 SWD runs up to 25 MHz with 3 ns edges (datasheet
Table 33). RESET_N stays Default. Docs and board drawing updated.
Other:
- board text added: "RMII, QSPI, SWD"
- board text removed: "RMII, ETH_REF_CLK, QSPI"

Commit message: layout: Setup rules, stackup etc.
Parts:
- removed R86: 47kΩ, Resistor_SMD:R_0402_1005Metric
- added R8: 100kΩ, Resistor_SMD:R_0402_1005Metric, F.Cu at (70.3, 254.9)
- added TP70: TP, TestPoint:TestPoint_Pad_D1.0mm, F.Cu at (76.5, 276.9)
- C89, C90, C91, C92: value 1nF -> 1.0nF
- R11, R28, R30: value 0 -> 0Ω
- R15: value 12M -> 12MΩ
- R23: value 1kΩ -> 127kΩ
- R42, R43: value 330Ω -> 1kΩ
- R52, R53: value 10 -> 10Ω
- R57, R58, R59: value 1k -> 1kΩ
- moved C1 272.7 mm to (25.4, 269.0)
- moved C42 272.7 mm to (29.3, 277.5)
- moved C43 272.7 mm to (25.4, 273.0)
- moved R35 272.7 mm to (28.5, 280.0)
- moved TP69 272.7 mm to (25.5, 280.5)
- moved C2 272.7 mm to (25.4, 271.0)
- moved TP6 272.7 mm to (25.5, 277.5)
- moved C28 252.2 mm to (151.4, 281.9), turned to 0 degrees
- moved R73 248.8 mm to (136.5, 277.4), turned to 0 degrees
- moved U10 247.6 mm to (34.7, 254.9)
- moved R74 246.8 mm to (136.5, 279.4)
- moved C24 239.8 mm to (41.9, 255.2)
- moved U15 237.9 mm to (150.1, 262.7), turned to 0 degrees
- moved R43 233.8 mm to (73.5, 278.4), turned to 0 degrees
- moved R76 233.1 mm to (128.7, 292.0), turned to 0 degrees
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Connections:
- net /IO/Digital Input/COOL_POUR renamed /IO/DI1/COOL_POUR
- net /IO/Digital Input1/COOL_POUR renamed /IO/DI2/COOL_POUR
- net /IO/Digital Input2/COOL_POUR renamed /IO/DI3/COOL_POUR
- net /IO/P24V_FIELD_EN renamed /MCU/P24V_FIELD_EN
- net /IO/RS485/P5V_RS485 renamed P5V_RS485
- net /MCU/USB_DM renamed /MCU/USB_D_N
- net /MCU/USB_DP renamed /MCU/USB_D_P
- net Net-(C19-Pad1) renamed /MCU/VDD_CORE
- net Net-(C57-Pad1) renamed /Ethernet & PoE/P12V0_FILTER
- net Net-(C78-Pad1) renamed /Power/P5V_RS485_FB_1
- net Net-(C84-Pad1) renamed /Power/P3V3_FB_1
- net Net-(C9-Pad1) renamed /MCU/V_SUPERCAP
- net Net-(R12-Pad1) renamed /Ethernet & PoE/P12V0_FB_1
- net Net-(U1-DCDC_LX) renamed /MCU/DCDC_LX
- net Net-(U1-VDD_SYS) renamed /MCU/VDD_SYS
- net Net-(U17-FB) renamed /Power/P5V_RS485_FB
- net Net-(U17-SW) renamed /Power/P5V_RS485_LX
- net Net-(U18-FB) renamed /Power/P3V3_FB
- net Net-(U3-XI) renamed /Ethernet & PoE/ETH_REF_CLK_PHY
- net Net-(U4-EROUT) renamed /Ethernet & PoE/POE_EROUT
- net Net-(U4-VDD) renamed /Ethernet & PoE/POE_VDD
- C33 pad 1: Net-(D17-K) -> /MCU/VDD_BAT
- D17 pad 2: (no net) -> /MCU/VDD_BAT
- D17 pad 3: Net-(D17-K) -> P3V3
- R23 pad 1: P3V3 -> P12V0
- R23 pad 2: /Ethernet & PoE/ETH_MDC -> Net-(U18-EN)
- R29 pad 2: Net-(J3-Pad01) -> Net-(J3-Pad1)
- R50 pad 1: Net-(D17-K) -> /MCU/VDD_BAT
- TP16 pad 1: Net-(D17-K) -> /MCU/VDD_BAT
- U1 pad 47: Net-(D17-K) -> /MCU/VDD_BAT
Routing:
- net /MCU/USB_D_P: track 0.00 -> 16.5 mm
- net GND: track 71.2 -> 55.3 mm, vias 91 -> 79
- net /MCU/USB_D_N: track 0.00 -> 15.9 mm
- net Net-(U15-SW2): track 12.7 -> 0.00 mm
- net /MCU/P24V_FIELD_EN: track 10.7 -> 0.00 mm, vias 2 -> 0
- net (no net): track 27.3 -> 18.1 mm
- net Net-(U15-SW1): track 8.14 -> 0.00 mm
- net Net-(U15-SS/ILIM): track 5.53 -> 0.00 mm
- net Net-(U15-SR): track 4.39 -> 0.00 mm
- net P12V0: track 8.46 -> 4.39 mm, vias 3 -> 2
- net P3V3: track 31.5 -> 30.8 mm, vias 21 -> 20

Commit message: hw: Layout: Routing complete.
Parts:
- removed TP14, TP24, TP25, TP31: TP, TestPoint:TestPoint_Pad_D1.0mm
- added TP71: TP, TestPoint:TestPoint_Pad_D1.0mm, F.Cu at (139.6, 82.4)
- moved TP69 259.4 mm to (159.4, 58.3)
- moved L2 258.3 mm to (134.9, 46.6), turned to -90 degrees
- moved TP6 257.9 mm to (165.6, 60.9)
- moved C28 256.6 mm to (36.0, 52.7), turned to 90 degrees
- moved TP62 252.8 mm to (138.4, 71.5)
- moved R73 252.5 mm to (33.6, 46.8)
- moved R74 252.3 mm to (41.6, 45.6), turned to 90 degrees
- moved TP68 251.6 mm to (37.1, 45.6)
- moved Q6 250.0 mm to (41.3, 51.5)
- moved R72 249.1 mm to (32.8, 48.9), turned to 90 degrees
- moved TP66 248.7 mm to (130.2, 75.3)
- moved TP63 248.0 mm to (132.3, 75.3)
- moved C83 245.4 mm to (122.1, 47.0), turned to -90 degrees
- moved TP50 244.9 mm to (39.8, 45.6)
- moved D22 242.3 mm to (48.8, 57.5), turned to 180 degrees
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Routing:
- net P12V0: track 4.39 -> 191.5 mm, vias 2 -> 14
- net GND: track 55.3 -> 167.4 mm, vias 79 -> 226
- net /MCU/RESET_N: track 0.00 -> 102.5 mm, vias 0 -> 3
- net /MCU/SWO: track 0.00 -> 94.8 mm, vias 0 -> 4
- net /MCU/P24V_FIELD_EN: track 0.00 -> 92.4 mm, vias 0 -> 2
- net /MCU/SWDIO: track 0.00 -> 91.0 mm, vias 0 -> 2
- net /MCU/DO1_ON: track 0.85 -> 91.9 mm, vias 1 -> 3
- net /MCU/SWDCLK: track 0.00 -> 90.4 mm, vias 0 -> 4
- net Net-(U9-IO1): track 0.00 -> 73.0 mm, vias 0 -> 2
- net /IO/DI_EN: track 4.74 -> 77.1 mm, vias 3 -> 5
- net P3V3: track 30.8 -> 102.1 mm, vias 20 -> 64
- net /MCU/DO2_ON: track 2.85 -> 73.3 mm, vias 1 -> 3
- net /Ethernet & PoE/ETH_MDIO: track 6.50 -> 69.8 mm
- net /Ethernet & PoE/ETH_REF_CLK_PHY: track 2.32 -> 65.2 mm, vias 1 -> 2
- net /MCU/VDD_BAT: track 0.00 -> 62.1 mm, vias 0 -> 2
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- added copper zone on In1.Cu, net /Ethernet & PoE/POE_VNEG
- added copper zone on In3.Cu, net /Ethernet & PoE/POE_VPOS
- added copper zone on In4.Cu, net /Ethernet & PoE/POE_VSS2
- added copper zone on F.Cu, net /IO/P24V0_FIELD_PROT
- added copper zone on In1.Cu, net GND
- added copper zone on F.Cu, net GND_FIELD
- added copper zone on In1.Cu, net GND_FIELD
- added copper zone on F.Cu, net P12V0
- added copper zone on F.Cu, net P24V0_FIELD
- added copper zone on In2.Cu, net P24V0_FIELD
- added copper zone on In2.Cu, net P3V3
- removed copper zone on F.Cu, net /IO/IN1_N
- removed copper zone on F.Cu, net /IO/IN1_P
- removed copper zone on F.Cu, net /IO/IN2_N
- removed copper zone on F.Cu, net /IO/IN2_P
- removed copper zone on F.Cu, net /IO/IN3_N
- removed copper zone on F.Cu, net /IO/IN3_P
- removed copper zone on F.Cu, net Net-(D12-A1)
- removed copper zone on F.Cu, net Net-(D20-A1)
- removed copper zone on F.Cu, net Net-(D21-A1)
