File: hw/poetato/poetato.kicad_sch (KiCad schematic)
At the start: 16 parts, among them M1 Light pipe, M10 Jumper, M11 Face Plate 1, M12 Face Plate 1, M13 Face Plate 2, M14 Face Plate 3, M15 Phoenix 12P plug, M16 Phoenix 4P plug, M2 Light pipe, M3 Light pipe, M4 Light pipe, M5 Light pipe, M6 Light pipe, M7 Light pipe, M8 Light pipe, M9 Enclosure

Commit message: hw: schematic and PCB update
- SE051C2 secure element, ENA tied to 3V3, RST_N to GND
- Epson TSX-3225 24 MHz and FC-135R 32.768 kHz crystals (replace NDK)
- LMR51420 RS-485 5 V buck (replaces TPS54202H)
- Field rail preload removed
- Datasheets updated to match (Würth connector added, unused
  NDK, TPS54202H, IHLP and Murata cap datasheets removed)

Co-Authored-By: Claude Opus 5.5 <noreply@anthropic.com>
Other:
- sheet IO ports: added DO1_ON, DO2_ON; removed DO1_EN, DO2_EN
- company: (none) -> Jonas Blixt <jonas@blxt.se>
- title: (none) -> PoEtato - Top level
Changed lines of the file:
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@@
 	(generator_version "10.0")
 	(paper "A3")
+	(title_block
+		(title "PoEtato - Top level")
+		(date "2026-10-08")
+		(rev "A (draft)")
+		(company "Jonas Blixt <jonas@blxt.se>")
+		(comment 1 "Copyright (c) 2026 Jonas Blixt. SPDX-License-Identifier: CERN-OHL-S-2.0")
+		(comment 2 "Licensed under CERN-OHL-S v2: https://ohwr.org/cern_ohl_s_v2.txt")
+		(comment 3 "Source location: https://github.com/jonasblixt/poetato")
+		(comment 4 "Status: draft, not released for manufacture")
+	)
 	(wire
 		(pts
@@
 			)
 		)
-		(pin "DO1_EN" input
+		(pin "DO1_ON" input
 			(at 203.2 54.61 180)
 			(effects
@@
 			)
 		)
-		(pin "DO2_EN" input
+		(pin "DO2_ON" input
 			(at 203.2 57.15 180)
 			(effects
@@
 	(sheet
 		(at 114.3 50.8)
-		(size 38.1 53.34)
+		(size 38.1 50.8)
 		(exclude_from_sim no)
 		(in_bom yes)
 		(on_board yes)
 		(dnp no)
-		(fields_autoplaced yes)
 		(stroke
 			(width 0.1524)
@@
 		)
 		(property "Sheetfile" "mcu.kicad_sch"
-			(at 114.3 102.1846 0)
+			(at 114.3 102.362 0)
 			(show_name no)
 			(do_not_autoplace no)
