File: hw/poetato/poetato.kicad_sch (KiCad schematic)
At the start: 16 parts, among them M1 Light pipe, M10 Jumper, M11 Face Plate 1, M12 Face Plate 1, M13 Face Plate 2, M14 Face Plate 3, M15 Phoenix 12P plug, M16 Phoenix 4P plug, M2 Light pipe, M3 Light pipe, M4 Light pipe, M5 Light pipe, M6 Light pipe, M7 Light pipe, M8 Light pipe, M9 Enclosure

Commit message: hw: fix local text collisions and add strap and BOM notes
- MCU: light-pipe note beside D14, TP64/TP65 references off the signal rows
- Ethernet: KSZ8081 strap summary (PHY address 1, RMII, auto-neg 100M),
  TP6 reference clear of POE_VDD
- IO: rating notes merged into the notes box
- DO: PhotoMOS note under K1
- Top level: frame and title around the BOM-only entries

Text and graphics only; ERC clean, netlist unchanged.
Other:
- note added: "Mechanical / BOM-only items"
Changed lines of the file:
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@@
+		)
+	)
+	(rectangle
+		(start 15.24 213.36)
+		(end 81.28 284.48)
+		(stroke
+			(width 0)
+			(type dash)
+		)
+		(fill
+			(type none)
+		)
+	)
+	(text "Mechanical / BOM-only items"
+		(exclude_from_sim no)
+		(at 17.78 218.44 0)
+		(effects
+			(font
+				(size 2.54 2.54)
+			)
+			(justify left)
 		)
 	)
