File: hw/poetato/rs485.kicad_sch (KiCad schematic)
At the start: 36 parts, among them J5 61300211121, Q7 FDV304P, Q8 FDV304P, U16 ISO3082, U17 TPS54202HDDCR

Commit message: hw: schematic and PCB update
- SE051C2 secure element, ENA tied to 3V3, RST_N to GND
- Epson TSX-3225 24 MHz and FC-135R 32.768 kHz crystals (replace NDK)
- LMR51420 RS-485 5 V buck (replaces TPS54202H)
- Field rail preload removed
- Datasheets updated to match (Würth connector added, unused
  NDK, TPS54202H, IHLP and Murata cap datasheets removed)

Co-Authored-By: Claude Opus 5.5 <noreply@anthropic.com>
Parts:
- added C93: ${Capacitance}, Capacitor_SMD:C_1206_3216Metric, symbol cap_mlcc_murata_GRM:GRM/C1206_4u7_50V_X7R_10%
- added R8, R97: 100kΩ, Resistor_SMD:R_0402_1005Metric, symbol res_chip_vishay_crcw:CRCW/R0402_100k0_1_63mW
- C76, C77: footprint Capacitor_SMD:C_0402_1005Metric -> Capacitor_SMD:C_0805_2012Metric; symbol cap_mlcc_murata_GRM:GRM/C0402_22u_10V_X5R_20% -> cap_mlcc_murata_GRM:GRM/C0805_22u_16V_X5R_20%; Part Number GRM158R61A226ME15 -> GRM21BR61C226ME44; Voltage 10V -> 16V
- C78: now not fitted
- C80: footprint Capacitor_SMD:C_0805_2012Metric -> Capacitor_SMD:C_1206_3216Metric; symbol cap_mlcc_murata_GRM:GRM/C0805_10u_50V_X5R_20% -> cap_mlcc_murata_GRM:GRM/C1206_4u7_50V_X7R_10%; Capacitance 10.0uF -> 4.7uF; Dielectric X5R -> X7R; Part Number GRM21BR61H106ME43 -> GRM31CR71H475KA12
- L3: value 22µH -> 10µH; symbol ind_power_vishay_ihlp:IHLP/L2020_22u_20_1A9 -> ind_power_vishay_ihlp:IHLP/L2020_10u_20_2A5; DCR 270mOhm Max -> 158mOhm Max; Inductance 22µH -> 10µH; Part Number IHLP2020CZER220M11 -> IHLP2020CZER100M01; Rated Current 1.9A -> 2.5A; SRF 10MHz -> N/A; Saturation Current 1.7A -> 4A
- R82: value 13.3kΩ -> 13.7kΩ; symbol res_chip_vishay_crcw:CRCW/R0402_13k3_1_63mW -> res_chip_vishay_crcw:CRCW/R0402_13k7_1_63mW; Part Number CRCW040213K3FKED -> CRCW040213K7FKED; Resistance 13.3kΩ -> 13.7kΩ
- R83: value 510kΩ -> 1MΩ; symbol res_chip_vishay_crcw:CRCW/R0402_510k0_1_63mW -> res_chip_vishay_crcw:CRCW/R0402_1M0_1_63mW; Part Number CRCW0402510KFKED -> CRCW04021M00FKED; Resistance 510kΩ -> 1MΩ
- U17: value TPS54202HDDCR -> LMR51420XDDCR; symbol dcdc:TPS54202HDDCR -> dcdc:LMR51420XDDCR; Part Number TPS54202HDDCR -> LMR51420XDDCR
Connections:
- net GND: now also R8.2
- net GND_FIELD: now also C93.2, R97.2
- net P24V0_FIELD: now also C93.1
- net RS485_R: now also R8.1
- net at R83.2, U17.5 (EN): now also R97.1
Other:
- note added: "Short to enable 120Ohm termination"
- company: (none) -> Jonas Blixt <jonas@blxt.se>
- title: (none) -> PoEtato - Isolated RS-485 and 5 V supply
- moved on the sheet: TP46
