File: hw/poetato/rs485.kicad_sch (KiCad schematic)
At the start: 39 parts, among them J5 61300211121, Q7 FDV304P, Q8 FDV304P, U16 ISO3082, U17 LMR51420XDDCR

Commit message: hw: RS485_RXD pull-up, 3V3 buck EN threshold, DC-only output rating
- R8 100 kOhm pull-up from RS485_RXD to P3V3 (review X3-1)
- 3V3 buck EN divider R23 127 kOhm / R87 20.5 kOhm (replaces R86
  47 kOhm): on at ~8.6 V, off at ~7.2 V (review Q-4)
- IO sheet note: outputs rated <= 30 V DC only (review E1-1)

Co-Authored-By: Claude Opus 5.5 <noreply@anthropic.com>
Connections:
- net GND: no longer R8.2
- net P3V3: now also R8.1
- net RS485_R: now also R8.2; no longer R8.1
Other:
- moved on the sheet: R8
Changed lines of the file:
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@@
 	(wire
 		(pts
-			(xy 96.52 162.56) (xy 96.52 170.18)
-		)
-		(stroke
-			(width 0)
-			(type default)
-		)
-	)
-	(wire
-		(pts
 			(xy 232.41 182.88) (xy 236.22 182.88)
 		)
@@
 	(wire
 		(pts
-			(xy 96.52 179.07) (xy 96.52 177.8)
-		)
-		(stroke
-			(width 0)
-			(type default)
-		)
-	)
-	(wire
-		(pts
 			(xy 196.85 234.95) (xy 196.85 236.22)
 		)
@@
 	(wire
 		(pts
+			(xy 82.55 162.56) (xy 96.52 162.56)
+		)
+		(stroke
+			(width 0)
+			(type default)
+		)
+	)
+	(wire
+		(pts
 			(xy 327.66 173.99) (xy 327.66 176.53)
 		)
@@
 	(wire
 		(pts
+			(xy 82.55 160.02) (xy 82.55 162.56)
+		)
+		(stroke
+			(width 0)
+			(type default)
+		)
+	)
+	(wire
+		(pts
 			(xy 184.15 133.35) (xy 184.15 129.54)
 		)
@@
 	(wire
 		(pts
+			(xy 82.55 148.59) (xy 82.55 152.4)
+		)
+		(stroke
+			(width 0)
+			(type default)
+		)
+	)
+	(wire
+		(pts
 			(xy 176.53 132.08) (xy 176.53 134.62)
 		)
@@
 	)
 	(symbol
-		(lib_id "power:GND")
-		(at 96.52 179.07 180)
-		(unit 1)
-		(body_style 1)
-		(exclude_from_sim no)
-		(in_bom yes)
-		(on_board yes)
-		(in_pos_files yes)
-		(dnp no)
-		(fields_autoplaced yes)
-		(property "Reference" "#PWR0176"
-			(at 96.52 182.626 0)
-			(hide yes)
-			(show_name no)
-			(do_not_autoplace no)
-			(effects
-				(font
-					(size 0.508 0.508)
-				)
-			)
-		)
-		(property "Value" "GND"
-			(at 96.52 181.61 0)
-			(show_name no)
-			(do_not_autoplace no)
-			(effects
-				(font
-					(size 0.762 0.762)
-				)
-			)
-		)
-		(property "Footprint" ""
-			(at 96.52 179.07 0)
-			(show_name no)
-			(do_not_autoplace no)
-			(effects
-				(font
-					(size 1.524 1.524)
-				)
-			)
-		)
-		(property "Datasheet" ""
-			(at 96.52 179.07 0)
-			(show_name no)
-			(do_not_autoplace no)
-			(effects
-				(font
-					(size 1.524 1.524)
-				)
-			)
-		)
-		(property "Description" ""
-			(at 96.52 179.07 0)
-			(hide yes)
-			(show_name no)
-			(do_not_autoplace no)
-			(effects
-				(font
-					(size 1.27 1.27)
-				)
-			)
-		)
-		(pin "1"
-		)
-		(instances
-			(project "poetato"
-				(path "/f0f504bb-124c-46e5-ad39-032d3dfa78b3/7f50897c-81bd-4425-95ed-f5153c9db421/21ef132d-889f-4c7f-901f-f28f90def5b6"
-					(reference "#PWR0176")
-					(unit 1)
-				)
-			)
-		)
-	)
-	(symbol
 		(lib_id "res_chip_vishay_crcw:CRCW/R0402_13k7_1_63mW")
 		(at 196.85 231.14 0)
@@
 	(symbol
 		(lib_id "res_chip_vishay_crcw:CRCW/R0402_100k0_1_63mW")
-		(at 96.52 173.99 0)
+		(at 82.55 156.21 0)
 		(unit 1)
 		(body_style 1)
@@
 		(fields_autoplaced yes)
 		(property "Reference" "R8"
-			(at 99.06 170.1799 0)
+			(at 85.09 152.3999 0)
 			(show_name no)
 			(do_not_autoplace no)
@@
 		)
 		(property "Value" "100kΩ"
-			(at 99.06 172.7199 0)
+			(at 85.09 154.9399 0)
 			(show_name no)
 			(do_not_autoplace no)
@@
 		)
 		(property "Footprint" "Resistor_SMD:R_0402_1005Metric"
-			(at 94.742 173.99 90)
+			(at 80.772 156.21 90)
 			(hide yes)
 			(show_name no)
@@
 		)
 		(property "Datasheet" ""
-			(at 96.52 173.99 0)
+			(at 82.55 156.21 0)
 			(hide yes)
 			(show_name no)
@@
 		)
 		(property "Description" "100kΩ, 1%, 63mW, TCR ±100ppm/K, EIA 0402"
-			(at 96.52 173.99 0)
+			(at 82.55 156.21 0)
 			(hide yes)
 			(show_name no)
@@
 		)
 		(property "Resistance" "100kΩ"
-			(at 96.52 173.99 0)
+			(at 82.55 156.21 0)
 			(hide yes)
 			(show_name yes)
@@
 		)
 		(property "Power" "63mW"
-			(at 99.06 175.2599 0)
+			(at 85.09 157.4799 0)
 			(show_name no)
 			(do_not_autoplace no)
@@
 		)
 		(property "Tolerance" "1%"
-			(at 99.06 177.7999 0)
+			(at 85.09 160.0199 0)
 			(show_name no)
 			(do_not_autoplace no)
@@
 		)
 		(property "T.C.R" "±100ppm/K"
-			(at 96.52 173.99 0)
+			(at 82.55 156.21 0)
 			(hide yes)
 			(show_name yes)
@@
 		)
 		(property "Manufacturer" "Vishay"
-			(at 96.52 173.99 0)
+			(at 82.55 156.21 0)
 			(hide yes)
 			(show_name yes)
@@
 		)
 		(property "Part Number" "CRCW0402100KFKED"
-			(at 96.52 173.99 0)
+			(at 82.55 156.21 0)
 			(hide yes)
 			(show_name yes)
@@
 					(unit 1)
 				)
+			)
+		)
+	)
+	(symbol
+		(lib_id "power:PxVx")
+		(at 82.55 148.59 0)
+		(unit 1)
+		(body_style 1)
+		(exclude_from_sim no)
+		(in_bom yes)
+		(on_board yes)
+		(in_pos_files yes)
+		(dnp no)
+		(fields_autoplaced yes)
+		(property "Reference" "#PWR0176"
+			(at 82.55 145.034 0)
+			(hide yes)
+			(show_name no)
+			(do_not_autoplace no)
+			(effects
+				(font
+					(size 0.508 0.508)
+				)
+			)
+		)
+		(property "Value" "P3V3"
+			(at 83.82 147.32 0)
+			(show_name no)
+			(do_not_autoplace no)
+			(effects
+				(font
+					(size 0.762 0.762)
+				)
+				(justify left)
+			)
+		)
+		(property "Footprint" ""
+			(at 82.55 148.59 0)
+			(show_name no)
+			(do_not_autoplace no)
+			(effects
+				(font
+					(size 1.524 1.524)
+				)
+			)
+		)
+		(property "Datasheet" ""
+			(at 82.55 148.59 0)
+			(show_name no)
+			(do_not_autoplace no)
+			(effects
+				(font
+					(size 1.524 1.524)
+				)
+			)
+		)
+		(property "Description" ""
+			(at 82.55 148.59 0)
+			(hide yes)
+			(show_name no)
+			(do_not_autoplace no)
+			(effects
+				(font
+					(size 1.27 1.27)
+				)
+			)
+		)
+		(pin "1"
+		)
+		(instances
+			(project "poetato"
+				(path "/f0f504bb-124c-46e5-ad39-032d3dfa78b3/7f50897c-81bd-4425-95ed-f5153c9db421/21ef132d-889f-4c7f-901f-f28f90def5b6"
+					(reference "#PWR0176")
+					(unit 1)
+				)

Commit message: hw: name test point nets, debug UART series 1 kOhm, DO notes
- Test point nets named (P12V0_FILTER, POE_VDD, POE_EROUT, VDD_SYS,
  VDD_BAT, VDD_CORE, DCDC_LX, V_SUPERCAP, loop injection nodes, ...)
  (review T4-1)
- R42 330 Ohm -> 1 kOhm on LPUART1_RXD, limits back-feed from a
  USB-UART cable on J4 into an unpowered board (review X2-1)
- DO sheet notes match arch §7: 1.5-2.1 A at a 24 V short (review H4-1)

Co-Authored-By: Claude Opus 5.5 <noreply@anthropic.com>
Connections:
- net P5V_RS485_FB: now reaches C78.2, R81.2, R82.1, U17.4 (FB)
- net P5V_RS485_FB_1: now reaches C78.1, R80.2, R81.1, TP28.1
- net P5V_RS485_LX: now reaches C75.1, L3.2, TP30.1, U17.2 (SW)
Other:
- note added: "TP30/TP32 For switch node measurement"
- moved on the sheet: C76, C77, L3, TP29
