File: hw/poetato/power.kicad_sch (KiCad schematic)
At the start: 60 parts, among them Q6 NTK3134N, T1 1308_750319693, U15 SN6507DGQR, U17 LMR51420XDDCR, U18 TPS563252DRLR

Commit message: hw: Layout: Routing complete.
Parts:
- removed TP24, TP25: TP, TestPoint:TestPoint_Pad_D1.0mm, symbol power:TP
